Commit message: 修改两轮底盘模型，添加四轮底盘模型及其控制

File: src/fishbot_description/urdf/fishbot_gazebo_four_wheeled_car.urdf (robot description, URDF)
Before this commit: robot fishbot, 17 links, 16 joints
Links:
- removed link caster_link
- removed link front_left_omni_base_link
- removed link front_left_omni_wheel_link
- removed link front_right_omni_base_link
- removed link front_right_omni_wheel_link
- removed link left_wheel_link
- removed link rear_left_omni_base_link
- removed link rear_left_omni_wheel_link
- removed link rear_right_omni_base_link
- removed link rear_right_omni_wheel_link
- removed link right_wheel_link
- added link front_left_steer_link, mass 0.2; visual cylinder length=0.06 radius=0.018
- added link front_left_wheel_link, mass 0.25; collision cylinder length=0.045 radius=0.06; visual cylinder length=0.045 radius=0.06
- added link front_right_steer_link, mass 0.2; visual cylinder length=0.06 radius=0.018
- added link front_right_wheel_link, mass 0.25; collision cylinder length=0.045 radius=0.06; visual cylinder length=0.045 radius=0.06
- added link rear_left_steer_link, mass 0.2; visual cylinder length=0.06 radius=0.018
- added link rear_left_wheel_link, mass 0.25; collision cylinder length=0.045 radius=0.06; visual cylinder length=0.045 radius=0.06
- added link rear_right_steer_link, mass 0.2; visual cylinder length=0.06 radius=0.018
- added link rear_right_wheel_link, mass 0.25; collision cylinder length=0.045 radius=0.06; visual cylinder length=0.045 radius=0.06
- link base_link: geometry collision box size=0.60 0.52 0.12; visual box size=0.60 0.52 0.12
Joints:
- removed joint caster_joint
- removed joint front_left_omni_base_joint
- removed joint front_left_omni_wheel_joint
- removed joint front_right_omni_base_joint
- removed joint front_right_omni_wheel_joint
- removed joint left_wheel_joint
- removed joint rear_left_omni_base_joint
- removed joint rear_left_omni_wheel_joint
- removed joint rear_right_omni_base_joint
- removed joint rear_right_omni_wheel_joint
- removed joint right_wheel_joint
- added joint front_left_steer_joint: type revolute, parent base_link, child front_left_steer_link, origin xyz=0.225 0.21 -0.016 rpy=0 0 0, axis 0 0 1, limit lower=-1.5708 upper=1.5708 effort=20.0 velocity=1.5
- added joint front_left_wheel_joint: type continuous, parent front_left_steer_link, child front_left_wheel_link, origin xyz=0 0 0 rpy=0 0 0, axis 0 1 0
- added joint front_right_steer_joint: type revolute, parent base_link, child front_right_steer_link, origin xyz=0.225 -0.21 -0.016 rpy=0 0 0, axis 0 0 1, limit lower=-1.5708 upper=1.5708 effort=20.0 velocity=1.5
- added joint front_right_wheel_joint: type continuous, parent front_right_steer_link, child front_right_wheel_link, origin xyz=0 0 0 rpy=0 0 0, axis 0 1 0
- added joint rear_left_steer_joint: type revolute, parent base_link, child rear_left_steer_link, origin xyz=-0.225 0.21 -0.016 rpy=0 0 0, axis 0 0 1, limit lower=-1.5708 upper=1.5708 effort=20.0 velocity=1.5
- added joint rear_left_wheel_joint: type continuous, parent rear_left_steer_link, child rear_left_wheel_link, origin xyz=0 0 0 rpy=0 0 0, axis 0 1 0
- added joint rear_right_steer_joint: type revolute, parent base_link, child rear_right_steer_link, origin xyz=-0.225 -0.21 -0.016 rpy=0 0 0, axis 0 0 1, limit lower=-1.5708 upper=1.5708 effort=20.0 velocity=1.5
- added joint rear_right_wheel_joint: type continuous, parent rear_right_steer_link, child rear_right_wheel_link, origin xyz=0 0 0 rpy=0 0 0, axis 0 1 0

File: src/fishbot_description/urdf/fishbot_gazebo_four_wheeled_car.urdf.xacro (robot description, xacro)
@@ -1,4 +1,5 @@
 <?xml version="1.0"?>
-<robot name="fishbot">
+<robot name="fishbot" xmlns:xacro="http://www.ros.org/wiki/xacro">
+  <xacro:arg name="controllers_file" default="/tmp/four_wheel_controllers.yaml"/>
   <!-- Robot Footprint -->
   <link name="base_footprint"/>
@@ -13,5 +14,5 @@
       <origin xyz="0 0 0.0" rpy="0 0 0"/>
       <geometry>
-		<box size="0.53 0.46 0.12"/>
+  		<box size="0.60 0.52 0.12"/>
       </geometry>
       <material name="blue">
@@ -22,5 +23,5 @@
       <origin xyz="0 0 0.0" rpy="0 0 0"/>
       <geometry>
-		<box size="0.53 0.46 0.12"/>
+		<box size="0.60 0.52 0.12"/>
       </geometry>
       <material name="blue">
@@ -88,358 +89,302 @@
       <origin xyz="0 0 0.02" />
   </joint>
-  <link name="left_wheel_link">
-      <visual>
-        <origin xyz="0 0 0" rpy="1.57079 0 0"/>
-        <geometry>
-          <cylinder length="0.04" radius="0.085"/>
-        </geometry>
-          <material name="black">
-            <color rgba="0.0 0.0 0.0 0.5" />
-          </material>
+  <!-- 四轮全向（四个独立转向 + 四个独立驱动） -->
+  <!-- 参数：左右轮距 0.42m，前后轮距 0.45m，轮半径 0.06m，转向偏移 y=0 -->
+  <!-- 前左转向电机（上层） -->
+  <link name="front_left_steer_link">
+      <visual>
+        <origin xyz="0 0 0.03" rpy="0 0 0"/>
+        <geometry>
+          <cylinder length="0.06" radius="0.018"/>
+        </geometry>
+        <material name="gray">
+          <color rgba="0.5 0.5 0.5 0.8" />
+        </material>
+      </visual>
+      <inertial>
+        <mass value="0.2"/>
+        <inertia ixx="0.0002" ixy="0" ixz="0" iyy="0.0002" iyz="0" izz="0.0002"/>
+      </inertial>
+  </link>
+  <joint name="front_left_steer_joint" type="revolute">
+      <parent link="base_link" />
+      <child link="front_left_steer_link" />
+      <origin xyz="0.225 0.21 -0.016" rpy="0 0 0" />
+      <axis xyz="0 0 1" />
+      <limit lower="-1.5708" upper="1.5708" effort="20.0" velocity="1.5"/>
+  </joint>
+  <link name="front_left_wheel_link">
+      <visual>
+        <origin xyz="0 0 0" rpy="1.57079 0 0"/>
+        <geometry>
+          <cylinder length="0.045" radius="0.06"/>
+        </geometry>
+        <material name="black">
+          <color rgba="0.0 0.0 0.0 0.7" />
+        </material>
       </visual>
       <collision>
         <origin xyz="0 0 0" rpy="1.57079 0 0"/>
         <geometry>
-          <cylinder length="0.04" radius="0.085"/>
-        </geometry>
-          <material name="black">
-            <color rgba="0.0 0.0 0.0 0.5" />
-          </material>
+          <cylinder length="0.045" radius="0.06"/>
+        </geometry>
       </collision>
       <inertial>
+        <mass value="0.25"/>
+        <inertia ixx="0.0003" ixy="0" ixz="0" iyy="0.0003" iyz="0" izz="0.0005"/>
+      </inertial>
+  </link>
+  <joint name="front_left_wheel_joint" type="continuous">
+      <parent link="front_left_steer_link" />
+      <child link="front_left_wheel_link" />
+      <origin xyz="0 0 0" rpy="0 0 0" />
+      <axis xyz="0 1 0" />
+  </joint>
+  <!-- 前右转向电机（上层） -->
+  <link name="front_right_steer_link">
+      <visual>
+        <origin xyz="0 0 0.03" rpy="0 0 0"/>
+        <geometry>
+          <cylinder length="0.06" radius="0.018"/>
+        </geometry>
+        <material name="gray">
+          <color rgba="0.5 0.5 0.5 0.8" />
+        </material>
+      </visual>
+      <inertial>
         <mass value="0.2"/>
-          <inertia ixx="0.000190416666667" ixy="0" ixz="0" iyy="0.0001904" iyz="0" izz="0.00036"/>
-        </inertial>
-  </link>
-  <link name="right_wheel_link">
-      <visual>
-        <origin xyz="0 0 0" rpy="1.57079 0 0"/>
-        <geometry>
-          <cylinder length="0.04" radius="0.085"/>
-        </geometry>
-          <material name="black">
-            <color rgba="0.0 0.0 0.0 0.5" />
-          </material>
+        <inertia ixx="0.0002" ixy="0" ixz="0" iyy="0.0002" iyz="0" izz="0.0002"/>
+      </inertial>
+  </link>
+  <joint name="front_right_steer_joint" type="revolute">
+      <parent link="base_link" />
+      <child link="front_right_steer_link" />
+      <origin xyz="0.225 -0.21 -0.016" rpy="0 0 0" />
+      <axis xyz="0 0 1" />
+      <limit lower="-1.5708" upper="1.5708" effort="20.0" velocity="1.5"/>
+  </joint>
+  <link name="front_right_wheel_link">
+      <visual>
+        <origin xyz="0 0 0" rpy="1.57079 0 0"/>
+        <geometry>
+          <cylinder length="0.045" radius="0.06"/>
+        </geometry>
+        <material name="black">
+          <color rgba="0.0 0.0 0.0 0.7" />
+        </material>
       </visual>
       <collision>
         <origin xyz="0 0 0" rpy="1.57079 0 0"/>
         <geometry>
-          <cylinder length="0.04" radius="0.085"/>
-        </geometry>
-          <material name="black">
-            <color rgba="0.0 0.0 0.0 0.5" />
-          </material>
+          <cylinder length="0.045" radius="0.06"/>
+        </geometry>
       </collision>
       <inertial>
-      <mass value="0.2"/>
-      <inertia ixx="0.000190416666667" ixy="0" ixz="0" iyy="0.0001904" iyz="0" izz="0.00036"/>
-    </inertial>
-  </link>
-  <joint name="left_wheel_joint" type="continuous">
+        <mass value="0.25"/>
+        <inertia ixx="0.0003" ixy="0" ixz="0" iyy="0.0003" iyz="0" izz="0.0005"/>
+      </inertial>
+  </link>
+  <joint name="front_right_wheel_joint" type="continuous">
+      <parent link="front_right_steer_link" />
+      <child link="front_right_wheel_link" />
+      <origin xyz="0 0 0" rpy="0 0 0" />
+      <axis xyz="0 1 0" />
+  </joint>
+  <!-- 后左转向电机（上层） -->
+  <link name="rear_left_steer_link">
+      <visual>
+        <origin xyz="0 0 0.03" rpy="0 0 0"/>
+        <geometry>
+          <cylinder length="0.06" radius="0.018"/>
+        </geometry>
+        <material name="gray">
+          <color rgba="0.5 0.5 0.5 0.8" />
+        </material>
+      </visual>
+      <inertial>
+        <mass value="0.2"/>
+        <inertia ixx="0.0002" ixy="0" ixz="0" iyy="0.0002" iyz="0" izz="0.0002"/>
+      </inertial>
+  </link>
+  <joint name="rear_left_steer_joint" type="revolute">
       <parent link="base_link" />
-      <child link="left_wheel_link" />
-      <origin xyz="-0.02 0.17 -0.06" />
+      <child link="rear_left_steer_link" />
+      <origin xyz="-0.225 0.21 -0.016" rpy="0 0 0" />
+      <axis xyz="0 0 1" />
+      <limit lower="-1.5708" upper="1.5708" effort="20.0" velocity="1.5"/>
+  </joint>
+  <link name="rear_left_wheel_link">
+      <visual>
+        <origin xyz="0 0 0" rpy="1.57079 0 0"/>
+        <geometry>
+          <cylinder length="0.045" radius="0.06"/>
+        </geometry>
+        <material name="black">
+          <color rgba="0.0 0.0 0.0 0.7" />
+        </material>
+      </visual>
+      <collision>
+        <origin xyz="0 0 0" rpy="1.57079 0 0"/>
+        <geometry>
+          <cylinder length="0.045" radius="0.06"/>
+        </geometry>
+      </collision>
+      <inertial>
+        <mass value="0.25"/>
+        <inertia ixx="0.0003" ixy="0" ixz="0" iyy="0.0003" iyz="0" izz="0.0005"/>
+      </inertial>
+  </link>
+  <joint name="rear_left_wheel_joint" type="continuous">
+      <parent link="rear_left_steer_link" />
+      <child link="rear_left_wheel_link" />
+      <origin xyz="0 0 0" rpy="0 0 0" />
       <axis xyz="0 1 0" />
   </joint>
-  <joint name="right_wheel_joint" type="continuous">
+  <!-- 后右转向电机（上层） -->
+  <link name="rear_right_steer_link">
+      <visual>
+        <origin xyz="0 0 0.03" rpy="0 0 0"/>
+        <geometry>
+          <cylinder length="0.06" radius="0.018"/>
+        </geometry>
+        <material name="gray">
+          <color rgba="0.5 0.5 0.5 0.8" />
+        </material>
+      </visual>
+      <inertial>
+        <mass value="0.2"/>
+        <inertia ixx="0.0002" ixy="0" ixz="0" iyy="0.0002" iyz="0" izz="0.0002"/>
+      </inertial>
+  </link>
+  <joint name="rear_right_steer_joint" type="revolute">
       <parent link="base_link" />
-      <child link="right_wheel_link" />
-      <origin xyz="-0.02 -0.17 -0.06" />
+      <child link="rear_right_steer_link" />
+      <origin xyz="-0.225 -0.21 -0.016" rpy="0 0 0" />
+      <axis xyz="0 0 1" />
+      <limit lower="-1.5708" upper="1.5708" effort="20.0" velocity="1.5"/>
+  </joint>
+  <link name="rear_right_wheel_link">
+      <visual>
+        <origin xyz="0 0 0" rpy="1.57079 0 0"/>
+        <geometry>
+          <cylinder length="0.045" radius="0.06"/>
+        </geometry>
+        <material name="black">
+          <color rgba="0.0 0.0 0.0 0.7" />
+        </material>
+      </visual>
+      <collision>
+        <origin xyz="0 0 0" rpy="1.57079 0 0"/>
+        <geometry>
+          <cylinder length="0.045" radius="0.06"/>
+        </geometry>
+      </collision>
+      <inertial>
+        <mass value="0.25"/>
+        <inertia ixx="0.0003" ixy="0" ixz="0" iyy="0.0003" iyz="0" izz="0.0005"/>
+      </inertial>
+  </link>
+  <joint name="rear_right_wheel_joint" type="continuous">
+      <parent link="rear_right_steer_link" />
+      <child link="rear_right_wheel_link" />
+      <origin xyz="0 0 0" rpy="0 0 0" />
       <axis xyz="0 1 0" />
   </joint>
-  <!-- 四个万象轮（前二后二，两段关节结构） -->
-  <!-- 前左万象轮基座（转向） -->
-  <link name="front_left_omni_base_link">
-      <visual>
-        <origin xyz="0 0 -0.015" rpy="0 0 0"/>
-        <geometry>
-          <cylinder length="0.03" radius="0.015"/>
-        </geometry>
-          <material name="gray">
-            <color rgba="0.5 0.5 0.5 0.8" />
-          </material>
-      </visual>
-      <inertial>
-        <mass value="0.05"/>
-          <inertia ixx="0.0001" ixy="0" ixz="0" iyy="0.0001" iyz="0" izz="0.0001"/>
-        </inertial>
-  </link>
-  <joint name="front_left_omni_base_joint" type="continuous">
-      <parent link="base_link" />
-      <child link="front_left_omni_base_link" />
-      <origin xyz="0.15 0.19 -0.015" />
-      <axis xyz="0 0 1" />
-  </joint>
-  <!-- 前左万象轮轮子（滚动） -->
-  <link name="front_left_omni_wheel_link">
-      <visual>
-        <origin xyz="0 0 0" rpy="1.57079 0 0"/>
-        <geometry>
-          <cylinder length="0.04" radius="0.05"/>
-        </geometry>
-          <material name="black">
-            <color rgba="0.0 0.0 0.0 0.5" />
-          </material>
-      </visual>
-      <collision>
-        <origin xyz="0 0 0" rpy="1.57079 0 0"/>
-        <geometry>
-          <cylinder length="0.04" radius="0.05"/>
-        </geometry>
-      </collision>
-      <inertial>
-        <mass value="0.1"/>
-          <inertia ixx="0.000190416666667" ixy="0" ixz="0" iyy="0.0001904" iyz="0" izz="0.00036"/>
-        </inertial>
-  </link>
-  <joint name="front_left_omni_wheel_joint" type="continuous">
-      <parent link="front_left_omni_base_link" />
-      <child link="front_left_omni_wheel_link" />
-      <origin xyz="0 0 -0.08" />
-      <axis xyz="1 0 0" />
-  </joint>
-  <!-- 前右万象轮基座（转向） -->
-  <link name="front_right_omni_base_link">
-      <visual>
-        <origin xyz="0 0 -0.015" rpy="0 0 0"/>
-        <geometry>
-          <cylinder length="0.03" radius="0.015"/>
-        </geometry>
-          <material name="gray">
-            <color rgba="0.5 0.5 0.5 0.8" />
-          </material>
-      </visual>
-      <inertial>
-        <mass value="0.05"/>
-          <inertia ixx="0.0001" ixy="0" ixz="0" iyy="0.0001" iyz="0" izz="0.0001"/>
-        </inertial>
-  </link>
-  <joint name="front_right_omni_base_joint" type="continuous">
-      <parent link="base_link" />
-      <child link="front_right_omni_base_link" />
-      <origin xyz="0.15 -0.19 -0.015" />
-      <axis xyz="0 0 1" />
-  </joint>
-  <!-- 前右万象轮轮子（滚动） -->
-  <link name="front_right_omni_wheel_link">
-      <visual>
-        <origin xyz="0 0 0" rpy="1.57079 0 0"/>
-        <geometry>
-          <cylinder length="0.04" radius="0.05"/>
-        </geometry>
-          <material name="black">
-            <color rgba="0.0 0.0 0.0 0.5" />
-          </material>
-      </visual>
-      <collision>
-        <origin xyz="0 0 0" rpy="1.57079 0 0"/>
-        <geometry>
-          <cylinder length="0.04" radius="0.05"/>
-        </geometry>
-      </collision>
-      <inertial>
-        <mass value="0.1"/>
-          <inertia ixx="0.000190416666667" ixy="0" ixz="0" iyy="0.0001904" iyz="0" izz="0.00036"/>
-        </inertial>
-  </link>
-  <joint name="front_right_omni_wheel_joint" type="continuous">
-      <parent link="front_right_omni_base_link" />
-      <child link="front_right_omni_wheel_link" />
-      <origin xyz="0 0 -0.08" />
-      <axis xyz="1 0 0" />
-  </joint>
-  <!-- 后左万象轮基座（转向） -->
-  <link name="rear_left_omni_base_link">
-      <visual>
-        <origin xyz="0 0 -0.015" rpy="0 0 0"/>
-        <geometry>
-          <cylinder length="0.03" radius="0.015"/>
-        </geometry>
-          <material name="gray">
-            <color rgba="0.5 0.5 0.5 0.8" />
-          </material>
-      </visual>
-      <inertial>
-        <mass value="0.05"/>
-          <inertia ixx="0.0001" ixy="0" ixz="0" iyy="0.0001" iyz="0" izz="0.0001"/>
-        </inertial>
-  </link>
-  <joint name="rear_left_omni_base_joint" type="continuous">
-      <parent link="base_link" />
-      <child link="rear_left_omni_base_link" />
-      <origin xyz="-0.15 0.19 -0.015" />
-      <axis xyz="0 0 1" />
-  </joint>
-  <!-- 后左万象轮轮子（滚动） -->
-  <link name="rear_left_omni_wheel_link">
-      <visual>
-        <origin xyz="0 0 0" rpy="1.57079 0 0"/>
-        <geometry>
-          <cylinder length="0.04" radius="0.05"/>
-        </geometry>
-          <material name="black">
-            <color rgba="0.0 0.0 0.0 0.5" />
-          </material>
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